File: ptn/pcb/ptn.kicad_sch (KiCad schematic)
At the start: 102 parts, among them IC1 ADP150AUJZ-3.3-R7, IC2 AZ1084CD-5.0TRG1, IC3 GRF5509, J1 TB002-500-04BE, J2 IO_BREAKOUT_CONN, J3 NRF_CONN, J4 Conn_01x04, J5 142-0701-801, J6 IO_CTRL_JP_BANK, SW1 SW_Push, U1 NCP1117-3.3_SOT223, U2 ADF4351, U3 MCP2551-I-SN, U4 STM32F103C8T6, Y1 SIT5000AICGE-33E0-25.000000X, Y2 16MHz

Commit message: PTN routing
Parts:
- removed J2: IO_BREAKOUT_CONN, Connector_PinHeader_2.54mm:PinHeader_2x12_P2.54mm_Vertical, symbol Connector_Generic:Conn_02x12_Counter_Clockwise
- removed J6: IO_CTRL_JP_BANK, Connector_PinHeader_2.54mm:PinHeader_2x12_P2.54mm_Vertical, symbol Connector_Generic:Conn_02x12_Counter_Clockwise
- added H1, H2, H3, H4: MountingHole_Pad, MountingHole:MountingHole_4.3mm_M4_Pad, symbol Mechanical:MountingHole_Pad
- added J2: ADC_IN_CONN, Connector_PinHeader_2.54mm:PinHeader_1x02_P2.54mm_Vertical, symbol Connector_Generic:Conn_01x02
- added J6: NRF_JUMPER_BANK, Connector_PinHeader_2.54mm:PinHeader_2x06_P2.54mm_Vertical, symbol Connector_Generic:Conn_02x06_Counter_Clockwise
- added J7: MCP2551_JUMPER_BANK, Connector_PinHeader_2.54mm:PinHeader_2x02_P2.54mm_Vertical, symbol Connector_Generic:Conn_02x02_Counter_Clockwise
- added J8: ADF_JUMPER_BANK, Connector_PinHeader_2.54mm:PinHeader_2x07_P2.54mm_Vertical, symbol Connector_Generic:Conn_02x07_Counter_Clockwise
- added J9: POWER_OUT_CONN, Connector_PinHeader_2.54mm:PinHeader_1x04_P2.54mm_Vertical, symbol Connector_Generic:Conn_01x04
Connections:
- net +3.3V: now also J9.2 (Pin_2)
- net +3.3VA: now also J9.3 (Pin_3)
- net +5V: now also J9.1 (Pin_1)
- net 12V_IN: now also J1.3; no longer J1.1
- net ADF4351_CE: now also J8.8 (Pin_8)
- net ADF4351_LD: now also J8.14 (Pin_14); no longer U4.19 (PB1)
- net ADF4351_MOSI: now also J8.10 (Pin_10)
- net ADF4351_MUXOUT: now also J8.12 (Pin_12); no longer U4.20 (PB2)
- net ADF4351_PDBRF: now also J8.13 (Pin_13)
- net ADF4351_SCK: now also J8.11 (Pin_11)
- net ADF4351_SSN: now also J8.9 (Pin_9)
- net CANH: now also J1.2; no longer J1.4
- net CANL: now also J1.1; no longer J1.3
- net GND: now also J1.4, H1.1, H2.1, H3.1, H4.1, J2.2 (Pin_2), J9.4 (Pin_4); no longer J1.2
- net MCP2551_CANRX: now also U3.4 (RXD), J7.3 (Pin_3)
- net MCP2551_CANTX: now also U3.1 (TXD), J7.4 (Pin_4)
- net NRF24L01P_CE: now also J6.11 (Pin_11)
- net NRF24L01P_IRQ: now also J6.1 (Pin_1), J6.12 (Pin_12)
- net NRF24L01P_MISO: now also J6.9 (Pin_9)
- net NRF24L01P_MOSI: now also J6.10 (Pin_10)
- net NRF24L01P_SCK: now also J6.8 (Pin_8)
- net NRF24L01P_SSN: now also J6.7 (Pin_7)
- net STM32_ADC1_IN0: now also J2.1 (Pin_1)
- net STM32_ADF_CE: now also J8.7 (Pin_7)
- net STM32_ADF_PDBRF: now also J8.2 (Pin_2)
- net STM32_CANRX: now also J7.2 (Pin_2); no longer U3.4 (RXD)
- net STM32_CANTX: now also J7.1 (Pin_1); no longer U3.1 (TXD)
- net STM32_NRF_CE: now also J6.2 (Pin_2)
- net STM32_SPI1_MOSI: now also J8.5 (Pin_5)
- net STM32_SPI1_SCK: now also J8.4 (Pin_4)
- net STM32_SPI1_SSN: now also J8.6 (Pin_6)
- net STM32_SPI2_MISO: now also J6.4 (Pin_4)
- net STM32_SPI2_MOSI: now also J6.3 (Pin_3)
- net STM32_SPI2_SCK: now also J6.5 (Pin_5)
- net STM32_SPI2_SSN: now also J6.6 (Pin_6)
- net STM32_USER_LED: now also U4.21 (PB10); no longer U4.2 (PC13)
- new net STM32_ADF_LD: J8.1 (Pin_1), U4.19 (PB1)
- new net STM32_ADF_MUXOUT: J8.3 (Pin_3), U4.20 (PB2)
Other:
- note added: "Mounting Holes"
- moved on the sheet: C10, C5, D1, D4, IC2, R9

Commit message: PTN routing part 3
Parts:
- R3: renamed from R2; footprint Resistor_SMD:R_0603_1608Metric -> Resistor_SMD:R_0402_1005Metric; Manufacturer_Part_Number RT0603BRE0750RL -> RC0402JR-0750RL; Mouser Part Number 603-RT0603BRE0750RL -> 603-RC0402JR-0750RL
- renumbered J3 to J2, J6 to J3, J2 to J4, J9 to J5, J7 to J6, J8 to J7, J4 to J8, J5 to J9, JP13 to JP1, L4 to L1, L1 to L2, L2 to L3, L3 to L4, R7 to R1, R9 to R10, R10 to R11, R11 to R12, R12 to R13, R13 to R14, R14 to R15, R15 to R16, R16 to R17, R1 to R2, R3 to R4, R4 to R5, R17 to R6, R5 to R7, R6 to R8, R8 to R9, U3 to U1, U1 to U2, U2 to U3

Commit message: finish all routing for ptn
Parts:
- removed C24: 10p, Capacitor_SMD:C_0402_1005Metric, symbol Device:C
- removed C27: 0.1u, Capacitor_SMD:C_0402_1005Metric, symbol Device:C
- renumbered C25 to C24, C26 to C25, C28 to C26, C29 to C27, C30 to C28, C31 to C29, C32 to C30, C33 to C31, C34 to C32, C35 to C33, C36 to C34, C37 to C35, C38 to C36, C39 to C37, C40 to C38, C41 to C39, C42 to C40, C43 to C41, C44 to C42, C45 to C43, C46 to C44, C47 to C45, C48 to C46, C49 to C47, C50 to C48, C51 to C49, C52 to C50, C53 to C51, C54 to C52, C55 to C53, C56 to C54, C57 to C55, C58 to C56, C59 to C57
