File: ptn/pcb/ptn.kicad_sch (KiCad schematic)
At the start: 107 parts, among them IC1 ADP150AUJZ-3.3-R7, IC2 AZ1084CD-5.0TRG1, IC3 GRF5509, J1 TB002-500-04BE, J2 NRF_CONN, J3 NRF_JUMPER_BANK, J4 ADC_IN_CONN, J5 POWER_OUT_CONN, J6 MCP2551_JUMPER_BANK, J7 ADF_JUMPER_BANK, J8 Conn_01x04, J9 142-0701-801, SW1 SW_Push, U1 MCP2551-I-SN, U2 NCP1117-3.3_SOT223, U3 ADF4351, U4 STM32F103C8T6, Y1 SIT5000AICGE-33E0-25.000000X, Y2 16MHz

Commit message: complete layout pending review
Parts:
- added J7: UART_CONN, Connector_PinHeader_2.54mm:PinHeader_1x02_P2.54mm_Vertical, symbol Connector_Generic:Conn_01x02
- renumbered J9 to J10, J7 to J8, J8 to J9, R11 to R10, R10 to R11
Connections:
- net STM32_USER_LED: now also U4.31 (PA10); no longer U4.21 (PB10)
- net STM32_USART3_RX: now reaches U4.22 (PB11)
- net STM32_USART3_RX: now also J7.2 (Pin_2)
- new net STM32_USART3_TX: J7.1 (Pin_1), U4.21 (PB10)
- no-connect marks 21 -> 19
Other:
- moved on the sheet: D4, R11

Commit message: Add another ADP150 LDO, improve T-line
Parts:
- removed J5: POWER_OUT_CONN, Connector_PinHeader_2.54mm:PinHeader_1x04_P2.54mm_Vertical, symbol Connector_Generic:Conn_01x04
- added C10, C13: 1u, Capacitor_SMD:C_0603_1608Metric, symbol Device:C
- added IC3: ADP150AUJZ-3.3-R7, project_footprint_library:SOT95P280X100-5N, symbol ADP150AUJZ-3_3-R7:ADP150AUJZ-3.3-R7
- added J5: POWER_OUT_CONN, Connector_PinHeader_2.54mm:PinHeader_1x05_P2.54mm_Vertical, symbol Connector_Generic:Conn_01x05
- renumbered C2 to C1, C10 to C11, C11 to C12, C12 to C14, C13 to C15, C14 to C16, C15 to C17, C16 to C18, C17 to C19, C1 to C2, C18 to C20, C19 to C21, C20 to C22, C21 to C23, C22 to C24, C23 to C25, C24 to C26, C25 to C27, C26 to C28, C27 to C29, C28 to C30, C29 to C31, C30 to C32, C31 to C33, C32 to C34, C33 to C35, C34 to C36, C35 to C37, C36 to C38, C37 to C39, C38 to C40, C39 to C41, C40 to C42, C41 to C43, C42 to C44, C43 to C45, C44 to C46, C45 to C47, C46 to C48, C47 to C49, C48 to C50, C49 to C51, C50 to C52, C51 to C53, C52 to C54, C53 to C55, C54 to C56, C55 to C57, C56 to C58, C57 to C59, C9 to C7, C7 to C8, C8 to C9, IC3 to IC4, J8 to J6, J6 to J7, J7 to J8
Connections:
- net +3.3V: now also J5.2 (Pin_2)
- net +3.3VA: now also J5.4 (Pin_4); no longer L1.1, R3.1
- net +5V: now also C10.1, IC3.1 (VIN), IC3.3 (EN), J5.1 (Pin_1)
- net GND: now also C10.2, C13.2, IC3.2 (GND), J5.5 (Pin_5)
- new net +3.3VA_VOUT: C13.1, IC3.5 (VOUT), J5.3 (Pin_3), L1.1, R3.1
Other:
- note removed: "No indicator LED added for 3.3VA, as it is only allocated for ADF4351."
- moved on the sheet: C1, C7, D2, D3, IC1, J3, J4, J6, J7, J8, R7, R8

Commit message: Layout review and optimization
Changed lines of the file:
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@@
 		)
 	)
-	(text_box "Tasks\n--------------------------\nAdd additional passive values for loop filter, matching, and amplifier to BOM.\nVerify MCU crystal.\nVerify MCU programming method (i.e., make sure SWD circuit is correct and enough).\nVerify MCU pins.\nDo complete review of schematic. COMPLETE REVIEW.\n"
+	(text_box "Tasks\n--------------------------\nBOM\nAdd additional passive values for loop filter, matching, and amplifier to BOM.\nVerify MCU programming method (i.e., make sure SWD circuit is correct and enough).\nAdd SW circuit to PCB, but DNP.\nFix NRF orientation.\nDo complete review of schematic. COMPLETE REVIEW.\n"
 		(exclude_from_sim no)
 		(at 850.9 -1.27 0)

Commit message: Add silkscreen, add SW, fix NRF orientation, add stm32 BOOT1
Parts:
- removed JP1: BOOT0_SEL, Connector_PinHeader_2.54mm:PinHeader_1x03_P2.54mm_Vertical, symbol Jumper:Jumper_3_Bridged12
- removed R17: 10k, Resistor_SMD:R_0603_1608Metric, symbol Device:R
- added C7: 1n, Capacitor_SMD:C_0402_1005Metric, symbol Device:C
- added J9: BOOT_SEL_JUMPER_BANK, Connector_PinHeader_2.54mm:PinHeader_2x03_P2.54mm_Vertical, symbol Connector_Generic:Conn_02x03_Counter_Clockwise
- added R19, R20: 10k, Resistor_SMD:R_0603_1608Metric, symbol Device:R
- added R3: ~, Resistor_SMD:R_0603_1608Metric, symbol Device:R
- added R7: 0R, Resistor_SMD:R_0603_1608Metric, symbol Device:R
- renumbered C9 to C10, C10 to C11, C11 to C12, C12 to C13, C13 to C14, C14 to C15, C15 to C16, C16 to C17, C17 to C18, C18 to C19, C19 to C20, C20 to C21, C21 to C22, C22 to C23, C23 to C24, C24 to C25, C25 to C26, C26 to C27, C27 to C28, C28 to C29, C29 to C30, C30 to C31, C31 to C32, C32 to C33, C33 to C34, C34 to C35, C35 to C36, C36 to C37, C37 to C38, C38 to C39, C39 to C40, C40 to C41, C41 to C42, C42 to C43, C43 to C44, C44 to C45, C45 to C46, C46 to C47, C47 to C48, C48 to C49, C49 to C50, C50 to C51, C51 to C52, C52 to C53, C53 to C54, C54 to C55, C55 to C56, C56 to C57, C57 to C58, C58 to C59, C59 to C60, C7 to C9, J9 to J10, J10 to J11, R8 to R10, R9 to R11, R10 to R12, R11 to R13, R12 to R14, R13 to R15, R14 to R16, R15 to R17, R16 to R18, R3 to R5, R5 to R6, R6 to R8, R7 to R9
Connections:
- net +3.3V: now also J9.1 (Pin_1), J9.6 (Pin_6)
- net ADF4351_RFOUTA+: now also C7.1
- net GND: now also J9.3 (Pin_3), J9.4 (Pin_4), R7.2; no longer R4.2
- net GRF5509_RFIN: now also C7.2
- net STM32_ADF_MUXOUT: now also U4.12 (PA2); no longer U4.20 (PB2)
- net STM32_BOOT0: now also R19.1
- net ADF4351_SW: now reaches U3.5 (SW)
- net ADF4351_SW: now also R3.1
- new net: R3.2, R4.2, R7.1
- new net: J9.5 (Pin_5), R20.1
- new net: J9.2 (Pin_2), R19.2
- new net STM32_BOOT1: R20.2, U4.20 (PB2)
- no-connect marks 19 -> 17
Other:
- note added: "BOOT0/BOOT1"
- note removed: "BOOT0"
- note removed: "Note: Check SW is needed or not."
- moved on the sheet: C3, C4, C58, C6, C60, C8, J10, L1, R4, R5, R6, Y2

Commit message: manufacturing ptn
Parts:
- added C13: 100p, Capacitor_SMD:C_0402_1005Metric, symbol Device:C
- added C14: 1n, Capacitor_SMD:C_0402_1005Metric, symbol Device:C
- added C16, C23: 120p, Capacitor_SMD:C_0402_1005Metric, symbol Device:C
- added C20: 0.1u, Capacitor_SMD:C_0402_1005Metric, symbol Device:C
- added L2: 1.9n, Inductor_SMD:L_0402_1005Metric, symbol Device:L
- added L3: 7.5n, Inductor_SMD:L_0402_1005Metric, symbol Device:L
- added R10, R11: 50R, Resistor_SMD:R_0402_1005Metric, symbol Device:R
- added R15, R16, R17, R18, R19: 10k, Resistor_SMD:R_0603_1608Metric, symbol Device:R
- added R8: 0R, Resistor_SMD:R_0402_1005Metric, symbol Device:R
- J10: renamed from J9; now left out of the parts list
- J11: renamed from J10; now left out of the parts list
- J2, J3, J4, J5, J6, J7, J8: now left out of the parts list
- R4: renamed from R3; now left out of the parts list
- R7: Manufacturer_Part_Number RCS04020000Z0ED -> RCS06030000Z0EA; Mouser Part Number 71-RCS04020000Z0ED -> 71-RCS06030000Z0EA
- renumbered C13 to C15, C14 to C17, C15 to C18, C16 to C19, C17 to C21, C18 to C22, C19 to C24, C20 to C25, C21 to C26, C22 to C27, C23 to C28, C24 to C29, C25 to C30, C26 to C31, C27 to C32, C28 to C33, C29 to C34, C30 to C35, C31 to C36, C32 to C37, C33 to C38, C34 to C39, C6 to C4, C35 to C40, C36 to C41, C37 to C42, C39 to C43, C41 to C44, C43 to C45, C45 to C46, C7 to C5, C51 to C50, C52 to C51, C53 to C52, C54 to C53, C38 to C54, C40 to C56, C42 to C57, C44 to C58, C46 to C59, C4 to C6, C50 to C60, C56 to C61, C57 to C62, C58 to C63, C59 to C64, C60 to C65, C5 to C7, J11 to J9, L2 to L4, L3 to L5, L4 to L6, R9 to R12, R10 to R13, R11 to R14, R5 to R2, R12 to R20, R14 to R21, R15 to R22, R16 to R23, R17 to R24, R18 to R25, R13 to R26, R19 to R27, R20 to R28, R2 to R3, R4 to R5, R8 to R9
Connections:
- net +3.3VA: now also R15.2, R16.2
- net +3.3VA_VOUT: now also C16.1, C20.1, C23.1, L3.1, R10.1
- net ADF4351_CE: now also R16.1
- net ADF4351_MOSI: now also R18.2
- net ADF4351_PDBRF: now also R15.1
- net ADF4351_SCK: now also R17.2
- net ADF4351_SSN: now also R19.2
- net GND: now also C16.2, C20.2, C23.2, R11.2, R17.1, R18.1, R19.1
- net GRF5509_RFIN: now also L2.2, R8.1; no longer C4.2
- net ADF4351_RFOUTA-: now reaches U3.13 (RF_OUT_A-)
- net ADF4351_RFOUTA-: now also C13.1, C14.1, L3.2, R10.2
- new net: C4.2, L2.1, R8.2
- new net: C13.2, C14.2, R11.1
- no-connect marks 17 -> 16
Other:
- moved on the sheet: C18, C21, C35, C36, C4, C5, C54, C56, C57, C58, C59, C60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

Commit message: exclude non-purchasable items from BOM
Parts:
- C40, C41, C42, C43, C45, C46, C47, C50, C51, C52: now left out of the parts list
- IC1, IC3: Mouser Part Number N/A -> 584-ADP150AUJZ-3.3R7
Changed lines of the file:
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@@
 		(unit 1)
 		(exclude_from_sim no)
-		(in_bom yes)
+		(in_bom no)
 		(on_board yes)
 		(dnp yes)
@@
 		(unit 1)
 		(exclude_from_sim no)
-		(in_bom yes)
+		(in_bom no)
 		(on_board yes)
 		(dnp yes)
@@
 			)
 		)
-		(property "Mouser Part Number" "N/A"
+		(property "Mouser Part Number" "584-ADP150AUJZ-3.3R7"
 			(at 161.29 637.16 0)
 			(effects
@@
 		(unit 1)
 		(exclude_from_sim no)
-		(in_bom yes)
+		(in_bom no)
 		(on_board yes)
 		(dnp yes)
@@
 		(unit 1)
 		(exclude_from_sim no)
-		(in_bom yes)
+		(in_bom no)
 		(on_board yes)
 		(dnp yes)
@@
 			)
 		)
-		(property "Mouser Part Number" "N/A"
+		(property "Mouser Part Number" "584-ADP150AUJZ-3.3R7"
 			(at 72.39 637.16 0)
 			(effects
@@
 		(unit 1)
 		(exclude_from_sim no)
-		(in_bom yes)
+		(in_bom no)
 		(on_board yes)
 		(dnp yes)
@@
 		(unit 1)
 		(exclude_from_sim no)
-		(in_bom yes)
+		(in_bom no)
 		(on_board yes)
 		(dnp yes)
@@
 		(unit 1)
 		(exclude_from_sim no)
-		(in_bom yes)
+		(in_bom no)
 		(on_board yes)
 		(dnp yes)
@@
 		(unit 1)
 		(exclude_from_sim no)
-		(in_bom yes)
+		(in_bom no)
 		(on_board yes)
 		(dnp yes)
@@
 		(unit 1)
 		(exclude_from_sim no)
-		(in_bom yes)
+		(in_bom no)
 		(on_board yes)
 		(dnp yes)
@@
 		(unit 1)
 		(exclude_from_sim no)
-		(in_bom yes)
+		(in_bom no)
 		(on_board yes)
 		(dnp yes)
